Commit message: Added a mimic link between j2 and j3.

File: urdf/sevenbot.urdf (robot description, URDF)
Before this commit: robot sevenbot, 8 links, 7 joints
Links:
- added link l2m
Joints:
- added joint j2m: type revolute, parent l2, child l2m, origin xyz=-0.12 0 0 rpy=0 0 0, axis 0 1 0, limit lower=0 upper=1.57 effort=100 velocity=100.0, mimic joint=j2 multiplier=-1
- joint j3: origin xyz=-0.12 0 0 rpy=0 0 0 -> (none); parent l2 -> l2m

Commit message: Succeeded in inporting angles from sevenbot.

File: urdf/sevenbot.urdf (robot description, URDF)
Before this commit: robot sevenbot, 9 links, 8 joints
Joints:
- joint j2: axis 0 1 0 -> 0 -1 0; origin xyz=0.03 0 0.075 rpy=0 0 0 -> xyz=0.03 0 0.075 rpy=0 2 0
- joint j2m: axis 0 1 0 -> 0 -1 0
- joint j3: origin (none) -> xyz=0 0 0 rpy=0 -1 0
